Commit message: First commit

File: ws/src/robot_description/urdf/bot.urdf.xacro (robot description, xacro)
@@ -1,4 +1,6 @@
 <?xml version="1.0" encoding="UTF-8"?>
-<robot name="bot_example" xmlns:xacro="http://www.ros.org/wiki/xacro">
+<robot name="bot" xmlns:xacro="http://www.ros.org/wiki/xacro">
+	<xacro:include filename="$(find robot_description)/urdf/bot_gazebo.xacro"/>
+	<xacro:include filename="$(find robot_description)/urdf/bot_ros2_control.xacro"/>
 	<xacro:property name="PI" value="3.1415926535897932384626433832795" />
 	<xacro:property name="effort" value="30.0" />
@@ -10,4 +12,13 @@
 		</inertial>
 	</xacro:macro>
+	<xacro:macro name="default_transmision" params="number">
+		<transmission name="transmission_${number}">
+			<plugin>transmission_interface/simpleTransmission</plugin>
+			<joint name="joint_${number}" role="joint1">
+				<mechanicalReduction>1.0</mechanicalReduction>
+			</joint>
+			<actuator name="motor_${number}" role="actuator1"/>
+		</transmission>
+	</xacro:macro>
 	<link name="world" />
 	<link name="base_link">
@@ -43,5 +54,5 @@
 		</visual>
 	</link>
-	<joint name="base_plate_joint" type="revolute">
+	<joint name="joint_1" type="revolute">
 		<parent link="base_link" />
 		<child link="base_plate" />
@@ -209,3 +220,7 @@
 	</sensor>
 </gazebo>
+	<xacro:default_transmision number="1"/>
+	<xacro:default_transmision number="2"/>
+	<xacro:default_transmision number="3"/>
+	<xacro:default_transmision number="4"/>
 </robot>

Commit message: feat: add simple action server

File: ws/src/robot_description/urdf/bot.urdf.xacro (robot description, xacro)
@@ -47,10 +47,10 @@
 				<mesh filename="package://robot_description/meshes/base_plate.STL" scale="0.01 0.01 0.01" />
 			</geometry>
-			<collision>
-				<geometry>
-					<mesh filename="package://robot_description/meshes/base_plate.STL" scale="0.01 0.01 0.01" />
-				</geometry>
-			</collision>
-		</visual>
+		</visual>
+		<collision>
+			<geometry>
+				<mesh filename="package://robot_description/meshes/base_plate.STL" scale="0.01 0.01 0.01" />
+			</geometry>
+		</collision>
 	</link>
 	<joint name="joint_1" type="revolute">

Commit message: feat: finish course

File: ws/src/robot_description/urdf/bot.urdf.xacro (robot description, xacro)
@@ -1,4 +1,5 @@
 <?xml version="1.0" encoding="UTF-8"?>
 <robot name="bot" xmlns:xacro="http://www.ros.org/wiki/xacro">
+	<xacro:arg name="is_sim" default="true"/>
 	<xacro:include filename="$(find robot_description)/urdf/bot_gazebo.xacro"/>
 	<xacro:include filename="$(find robot_description)/urdf/bot_ros2_control.xacro"/>

File: ws/src/robot_description/urdf/bot_ros2_control.xacro (robot description, xacro)
@@ -3,7 +3,24 @@
     <xacro:property name="PI" value="3.1415926535897932384626433832795" />
     <ros2_control type="system" name="RobotSystem">
-        <hardware>
-            <plugin>gazebo_ros2_control/GazeboSystem</plugin>
-        </hardware>
+        <xacro:if value="${arg is_sim}">
+            <hardware>
+                <plugin>gazebo_ros2_control/GazeboSystem</plugin>
+            </hardware>
+            <joint name="joint_5">
+                <param name="mimic">joint_4</param>
+                <param name="multiplier">-1</param>
+                <command_interface name="position">
+                    <param name="min">0.0</param>
+                    <param name="max">${PI/2}</param>
+                </command_interface>
+                <state_interface name="position"/>
+            </joint>
+        </xacro:if>
+        <xacro:unless value="${arg is_sim}">
+            <hardware>
+                <plugin>bot_controller::BotInterface</plugin>
+                <param name="port">/dev/ttyACM0</param>
+            </hardware>
+        </xacro:unless>
         <joint name="joint_1">
             <command_interface name="position">
@@ -34,13 +51,4 @@
             <state_interface name="position"/>
         </joint>
-        <joint name="joint_5">
-            <param name="mimic">joint_4</param>
-            <param name="multiplier">-1</param>
-            <command_interface name="position">
-                <param name="min">0.0</param>
-                <param name="max">${PI/2}</param>
-            </command_interface>
-            <state_interface name="position"/>
-        </joint>
         </ros2_control>
 </robot>
